File: vdg.kicad_sch (KiCad schematic)
At the start: 3 parts, among them IC12 MC6847, IC13 74LS273N

Commit message: remove video
Parts:
- removed IC13: 74LS273N, Package_DIP:DIP-20_W7.62mm, symbol 74xx:74LS273
- added J1: Board interconnect female, Connector_PinHeader_2.54mm:PinHeader_2x10_P2.54mm_Vertical, symbol Connector_Generic:Conn_02x10_Odd_Even
- added J2: Video Output, Connector_PinHeader_2.54mm:PinHeader_1x05_P2.54mm_Vertical, symbol Connector:Conn_01x05_Pin
Connections:
- net +5V: now also J1.1 (Pin_1), J2.2 (Pin_2)
- net CSS: now also J1.19 (Pin_19)
- net DA0: now also J1.6 (Pin_6)
- net DO0: now also J1.3 (Pin_3)
- net DO1: now also J1.5 (Pin_5)
- net DO2: now also J1.7 (Pin_7)
- net DO3: now also J1.9 (Pin_9)
- net DO4: now also J1.11 (Pin_11)
- net DO5: now also J1.13 (Pin_13)
- net DO6: now also J1.15 (Pin_15)
- net DO7: now also J1.17 (Pin_17)
- net GM0: now also J1.14 (Pin_14)
- net GM1: now also J1.12 (Pin_12)
- net GM2: now also J1.10 (Pin_10)
- net GND: now also J1.4 (Pin_4), J2.5 (Pin_5)
- net ~{A}/G: now also J1.20 (Pin_20)
- net ~{HS}: now also J1.8 (Pin_8)
- net ~{RAS0}: now also J1.16 (Pin_16)
- new net -5V: J1.2 (Pin_2)
- new net BIAS: J2.1 (Pin_1)
- new net VCLK: J1.18 (Pin_18)
- new net VID OUT: J2.4 (Pin_4)
- no-connect marks 13 -> 14
