File: Dragon32.kicad_pcb (KiCad board)
At the start: 2 copper layers, 253 x 169.1 mm, 142 parts, among them IC1 4164, IC15 MC6883, IC16 74LS244N, IC17 27C256, IC18 74LS08, IC19 MC6809E, IC2 4164, IC20 MC14529B, IC24 74LS244N, IC25 LM393P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

Commit message: add third pia
Parts:
- added C2: 10uF, Capacitor_THT:CP_Radial_D5.0mm_P2.50mm, F.Cu at (158.9, 132.4)
- added IC10: MC14053, Package_DIP:DIP-16_W7.62mm, F.Cu at (134.5, 143.9)
- added IC9: MC6821, Package_DIP:DIP-40_W15.24mm, F.Cu at (163.5, 84.1)
- J2: value Board Interconnect Female -> Video Interconnect Female; footprint Connector_PinSocket_2.54mm:PinSocket_2x11_P2.54mm_Vertical -> Connector_PinSocket_2.54mm:PinSocket_2x12_P2.54mm_Vertical
- moved C42 21.9 mm to (225.8, 185.8)
Connections:
- J2 pad 21: unconnected-(J2-Pin_21-Pad21) -> INV
Routing:
- net P2: track 70.1 -> 201.0 mm, vias 2 -> 7
- net GND: track 1774.3 -> 1879.4 mm, vias 56 -> 58
- net D7: track 342.9 -> 425.8 mm, vias 7 -> 8
- net R/~{W}: track 252.9 -> 335.4 mm, vias 7 -> 8
- net D6: track 362.2 -> 438.0 mm, vias 11 -> 13
- net ~{A}/S: track 0.00 -> 73.3 mm, vias 0 -> 1
- net P-~{A}/S: track 0.00 -> 72.7 mm, vias 0 -> 3
- net INV: track 0.00 -> 65.8 mm, vias 0 -> 1
- net ~{INT}/EXT: track 0.00 -> 65.3 mm, vias 0 -> 4
- net P-~{INT}/EXT: track 0.00 -> 63.4 mm, vias 0 -> 3
- net P-INV: track 0.00 -> 62.8 mm, vias 0 -> 2
- net C-A: track 0.00 -> 62.5 mm, vias 0 -> 2
- net E: track 268.0 -> 328.8 mm, vias 8 -> 9
- net C-B: track 0.00 -> 55.1 mm, vias 0 -> 2
- net C-C: track 0.00 -> 52.5 mm, vias 0 -> 2
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