File: Dragon32.kicad_pcb (KiCad board)
At the start: 2 copper layers, 253 x 169.1 mm, 171 parts, among them IC1 4164, IC10 74ACT138, IC15 MC6883, IC16 74LS244N, IC17 27C256, IC18 74LS08, IC19 MC6809E, IC2 4164, IC20 MC14529B, IC24 74LS244N, IC25 LM393P, IC26 MC6821, IC3 4164, IC31 74LS02N, IC33 74ACT138N, IC34 MC14050BCP, IC35 MC6821, IC36 74LS132, IC37 GAL, IC38 74LS08, IC39 74LS04, IC4 4164, IC5 4164, IC6 4164, IC7 4164, IC8 4164, J1 Video Output Female, J2 Board Interconnect Female, J3 Conn_02x08_Odd_Even, J4 PSG Audio, J5 Config, SW1 RESET, U1 MAX3232, U12 M6551, U2 GAL22V10

Commit message: include CUPL for keyboard GAL
Parts:
- moved C43 2.58 mm to (104.1, 163.7)
- moved R31 2.31 mm to (120.3, 116.6)
- moved D7 0.13 mm to (124.4, 150.9)
Connections:
- IC38 pad 11: BC11 -> unconnected-(IC38-Pad11)
- IC38 pad 6: BDIR1 -> unconnected-(IC38-Pad6)
- IC39 pad 11: ~{P1d} -> GND
- IC39 pad 13: ~{P1c} -> ~{P1d}
- J2 pad 2: unconnected-(J2-Pin_2-Pad2) -> ~{RES}
- J2 pad 21: E -> GND
- J3 pad 10: unconnected-(J3-Pin_10-Pad10) -> ~{P1c}
- J3 pad 2: unconnected-(J3-Pin_2-Pad2) -> A0
- J3 pad 4: unconnected-(J3-Pin_4-Pad4) -> A1
- J3 pad 6: unconnected-(J3-Pin_6-Pad6) -> A2
- J3 pad 8: unconnected-(J3-Pin_8-Pad8) -> A3
Routing:
- net A3: track 241.8 -> 404.1 mm, vias 8 -> 11
- net A2: track 277.9 -> 386.7 mm, vias 11 -> 13
- net A1: track 381.6 -> 462.0 mm, vias 12 -> 13
- net A0: track 326.8 -> 396.7 mm, vias 8 -> 10
- net E: track 619.5 -> 593.8 mm, vias 13 -> 12
- net ~{P1c}: track 270.1 -> 293.1 mm, vias 5 -> 6
- net ~{RES}: track 553.8 -> 574.3 mm, vias 9 -> 10
- net GND: track 803.6 -> 788.8 mm, vias 299 -> 305
- net Net-(IC25A-+): track 30.4 -> 24.3 mm, vias 2 -> 1
- net ~{P1d}: track 261.8 -> 267.7 mm
- net +5V: track 1644.8 -> 1640.9 mm
- net PC0: track 143.0 -> 140.9 mm, vias 7 -> 5
- net PB2: track 126.6 -> 128.6 mm
- net CASS: track 58.9 -> 61.0 mm
- net Net-(D7-K): track 16.7 -> 14.6 mm
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Other:
- board text added: "Revision 3.3c"
- board text removed: "Revision 3.3b"
