File: mpu.kicad_sch (KiCad schematic)
At the start: 14 parts, among them IC19 MC6809E, SW1 RESET

Commit message: refresh BOM
Parts:
- IC19: SA2120 Sheet 1 -> (none)
Changed lines of the file:
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@@
-			)
-		)
-		(property "SA2120" "Sheet 1"
-			(at 168.148 94.234 0)
-			(effects
-				(font
-					(size 1.27 1.27)
-				)
-				(hide yes)
 			)
 		)

Commit message: align versions
Other:
- title: (none) -> Dragon CPU UK Revised
Changed lines of the file:
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@@
 	(paper "A3")
 	(title_block
-		(date "2023-05-25")
-		(rev "3.0")
+		(title "Dragon CPU UK Revised")
+		(date "2025-10-05")
+		(rev "3.3")
+		(comment 1 "Redesign by Julian Brown")
 		(comment 2 "Reposition dram and buffer")
 	)
