File: Dragon32.kicad_sch (KiCad schematic)
At the start: 6 parts, among them IC25 LM393P, IC31 74LS02N, J5 Config

Commit message: refresh BOM
Parts:
- IC25: LCSC (none) -> C5209
- IC31: LCSC (none) -> C22374091; SA2120 Sheet 1 (spare) -> (none)
Changed lines of the file:
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@@
+			)
+		)
+		(property "LCSC" "C5209"
+			(at 98.425 51.054 0)
+			(effects
+				(font
+					(size 1.27 1.27)
+				)
+				(hide yes)
 			)
 		)
@@
 			)
 		)
-		(property "SA2120" "Sheet 1 (spare)"
+		(property "LCSC" "C22374091"
 			(at 65.913 49.911 0)
 			(effects

Commit message: align versions
Other:
- company: Dragon Data -> (none)
- title: Dragon 32 CPU UK PAL -> Dragon CPU UK Revised
Changed lines of the file:
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@@
 	(paper "A3")
 	(title_block
-		(title "Dragon 32 CPU UK PAL")
-		(date "2023-05-25")
-		(rev "3.0")
-		(company "Dragon Data")
-		(comment 1 "Recreation by Julian Brown")
+		(title "Dragon CPU UK Revised")
+		(date "2025-10-05")
+		(rev "3.3")
+		(comment 1 "Redesign by Julian Brown")
 	)
 	(junction
