File: audio.kicad_sch (KiCad schematic)
At the start: 8 parts, among them IC38 74LS08, IC39 74LS04, J4 PSG Audio

Commit message: refresh BOM
Parts:
- IC38: LCSC (none) -> C22394768
- IC39: LCSC (none) -> C22374093
Changed lines of the file:
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@@
+			)
+		)
+		(property "LCSC" "C22394768"
+			(at 162.56 88.9 0)
+			(effects
+				(font
+					(size 1.27 1.27)
+				)
+				(hide yes)
 			)
 		)
@@
 			)
 		)
+		(property "LCSC" "C22394768"
+			(at 162.56 137.16 0)
+			(effects
+				(font
+					(size 1.27 1.27)
+				)
+				(hide yes)
+			)
+		)
 		(pin "1"
 		)
@@
 			)
 		)
+		(property "LCSC" "C22394768"
+			(at 156.21 175.26 0)
+			(effects
+				(font
+					(size 1.27 1.27)
+				)
+				(hide yes)
+			)
+		)
 		(pin "1"
 		)
@@
 			)
 		)
+		(property "LCSC" "C22374093"
+			(at 270.51 156.21 0)
+			(effects
+				(font
+					(size 1.27 1.27)
+				)
+				(hide yes)
+			)
+		)
 		(pin "12"
 		)
@@
 			)
 		)
+		(property "LCSC" "C22374093"
+			(at 270.51 142.24 0)
+			(effects
+				(font
+					(size 1.27 1.27)
+				)
+				(hide yes)
+			)
+		)
 		(pin "12"
 		)
@@
 			)
 		)
+		(property "LCSC" "C22394768"
+			(at 162.56 102.87 0)
+			(effects
+				(font
+					(size 1.27 1.27)
+				)
+				(hide yes)
+			)
+		)
 		(pin "1"
 		)
@@
 			)
 		)
+		(property "LCSC" "C22374093"
+			(at 138.43 86.36 0)
+			(effects
+				(font
+					(size 1.27 1.27)
+				)
+				(hide yes)
+			)
+		)
 		(pin "12"
 		)
@@
 		)
 		(property "Description" "Hex Inverter"
+			(at 270.51 115.57 0)
+			(effects
+				(font
+					(size 1.27 1.27)
+				)
+				(hide yes)
+			)
+		)
+		(property "LCSC" "C22374093"
 			(at 270.51 115.57 0)
 			(effects
@@
 			)
 		)
+		(property "LCSC" "C22374093"
+			(at 134.62 175.26 0)
+			(effects
+				(font
+					(size 1.27 1.27)
+				)
+				(hide yes)
+			)
+		)
 		(pin "12"
 		)
@@
 		)
 		(property "Description" ""
+			(at 162.56 123.19 0)
+			(effects
+				(font
+					(size 1.27 1.27)
+				)
+				(hide yes)
+			)
+		)
+		(property "LCSC" "C22394768"
 			(at 162.56 123.19 0)
 			(effects
@@
 			)
 		)
+		(property "LCSC" "C22374093"
+			(at 138.43 120.65 0)
+			(effects
+				(font
+					(size 1.27 1.27)
+				)
+				(hide yes)
+			)
+		)
 		(pin "12"
 		)
@@
 			(at 270.51 128.27 0)
 			(effects
+				(font
+					(size 1.27 1.27)
+				)
+				(hide yes)
+			)
+		)
+		(property "LCSC" "C22374093"
+			(at 270.51 128.27 0)
+			(effects

Commit message: include CUPL for keyboard GAL
Connections:
- net ~{P1c} is gone; now on net ~{P1d}: IC39.13
- net GND: now also IC39.11
- net ~{P1d}: no longer IC39.11
- net BC11: no longer names the net of IC38.11
- net BDIR1: no longer names the net of IC38.6
- no-connect marks 9 -> 11

Commit message: align versions
Other:
- title: (none) -> Dragon CPU UK Revised
Changed lines of the file:
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@@
 	(generator_version "9.0")
 	(paper "A4")
+	(title_block
+		(title "Dragon CPU UK Revised")
+		(date "2025-10-05")
+		(rev "3.3")
+		(comment 1 "Redesign by Julian Brown")
+	)
 	(junction
 		(at 139.7 31.75)
