File: audio.kicad_sch (KiCad schematic)
At the start: 8 parts, among them IC38 74LS08, IC39 74LS04, J4 PSG Audio

Commit message: update to keyboard switch option
Parts:
- IC38: LCSC (none) -> C22394768
- IC39: LCSC (none) -> C22374093
Connections:
- net ~{P1c} is gone; now on net ~{P1d}: IC39.13
- net GND: now also IC39.11
- net ~{P1d}: no longer IC39.11
- net BC11: no longer names the net of IC38.11
- net BDIR1: no longer names the net of IC38.6
- no-connect marks 9 -> 11
Other:
- title: (none) -> Dragon CPU UK Revised
