File: serial.kicad_sch (KiCad schematic)
At the start: 12 parts, among them U1 MAX3232, U12 M6551

Commit message: update to keyboard switch option
Parts:
- C3: value 100n -> 100nF; footprint Capacitor_SMD:C_0805_2012Metric_Pad1.18x1.45mm_HandSolder -> PCM_Capacitor_SMD_AKL:C_0805_2012Metric_Pad1.18x1.45mm_HandSolder; LCSC (none) -> C1711
- C5, C6, C7, C8, C9: footprint Capacitor_SMD:C_0805_2012Metric_Pad1.18x1.45mm_HandSolder -> PCM_Capacitor_SMD_AKL:C_0805_2012Metric_Pad1.18x1.45mm_HandSolder; DigiKey 311-1140-1-ND -> (none); LCSC MBK0805X7R104K500NT -> C1711
- R10, R11: LCSC (none) -> C17673
Other:
- title: (none) -> Dragon CPU UK Revised
Changed lines of the file:
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@@
 	(generator_version "9.0")
 	(paper "A4")
+	(title_block
+		(title "Dragon CPU UK Revised")
+		(date "2025-10-05")
+		(rev "3.3")
+		(comment 1 "Redesign by Julian Brown")
+	)
 	(junction
 		(at 226.06 24.13)
@@
 			)
 		)
+		(property "LCSC" "C17673"
+			(at 250.19 133.35 90)
+			(effects
+				(font
+					(size 1.27 1.27)
+				)
+				(hide yes)
+			)
+		)
 		(pin "1"
 		)
@@
 			)
 		)
-		(property "Footprint" "Capacitor_SMD:C_0805_2012Metric_Pad1.18x1.45mm_HandSolder"
+		(property "Footprint" "PCM_Capacitor_SMD_AKL:C_0805_2012Metric_Pad1.18x1.45mm_HandSolder"
 			(at 201.93 109.22 0)
 			(effects
@@
 			)
 		)
-		(property "DigiKey" "311-1140-1-ND"
+		(property "DigiKey" ""
 			(at 201.93 109.22 0)
 			(effects
@@
 			)
 		)
-		(property "LCSC" "MBK0805X7R104K500NT"
+		(property "LCSC" "C1711"
 			(at 201.93 109.22 0)
 			(effects
@@
 			)
 		)
-		(property "Footprint" "Capacitor_SMD:C_0805_2012Metric_Pad1.18x1.45mm_HandSolder"
+		(property "Footprint" "PCM_Capacitor_SMD_AKL:C_0805_2012Metric_Pad1.18x1.45mm_HandSolder"
 			(at 175.26 80.01 0)
 			(effects
@@
 			)
 		)
-		(property "DigiKey" "311-1140-1-ND"
+		(property "DigiKey" ""
 			(at 175.26 80.01 0)
 			(effects
@@
 			)
 		)
-		(property "LCSC" "MBK0805X7R104K500NT"
+		(property "LCSC" "C1711"
 			(at 175.26 80.01 0)
 			(effects
@@
 			)
 		)
-		(property "Footprint" "Capacitor_SMD:C_0805_2012Metric_Pad1.18x1.45mm_HandSolder"
+		(property "Footprint" "PCM_Capacitor_SMD_AKL:C_0805_2012Metric_Pad1.18x1.45mm_HandSolder"
 			(at 157.48 92.71 0)
 			(effects
@@
 			)
 		)
-		(property "DigiKey" "311-1140-1-ND"
+		(property "DigiKey" ""
 			(at 157.48 92.71 0)
 			(effects
@@
 			)
 		)
-		(property "LCSC" "MBK0805X7R104K500NT"
+		(property "LCSC" "C1711"
 			(at 157.48 92.71 0)
 			(effects
@@
 			)
 		)
-		(property "Value" "100n"
+		(property "Value" "100nF"
 			(at 222.25 26.67 90)
 			(effects
@@
 			)
 		)
-		(property "Footprint" "Capacitor_SMD:C_0805_2012Metric_Pad1.18x1.45mm_HandSolder"
+		(property "Footprint" "PCM_Capacitor_SMD_AKL:C_0805_2012Metric_Pad1.18x1.45mm_HandSolder"
 			(at 219.71 24.13 0)
 			(effects
@@
 		(property "Description" ""
 			(at 219.71 24.13 0)
+			(effects
+				(font
+					(size 1.27 1.27)
+				)
+				(hide yes)
+			)
+		)
+		(property "LCSC" "C1711"
+			(at 219.71 24.13 90)
 			(effects
 				(font
@@
 			)
 		)
-		(property "Footprint" "Capacitor_SMD:C_0805_2012Metric_Pad1.18x1.45mm_HandSolder"
+		(property "Footprint" "PCM_Capacitor_SMD_AKL:C_0805_2012Metric_Pad1.18x1.45mm_HandSolder"
 			(at 201.93 101.6 0)
 			(effects
@@
 			)
 		)
-		(property "DigiKey" "311-1140-1-ND"
+		(property "DigiKey" ""
 			(at 201.93 101.6 0)
 			(effects
@@
 			)
 		)
-		(property "LCSC" "MBK0805X7R104K500NT"
+		(property "LCSC" "C1711"
 			(at 201.93 101.6 0)
 			(effects
@@
 			)
 		)
+		(property "LCSC" "C17673"
+			(at 250.19 137.16 90)
+			(effects
+				(font
+					(size 1.27 1.27)
+				)
+				(hide yes)
+			)
+		)
 		(pin "1"
 		)
@@
 			)
 		)
-		(property "Footprint" "Capacitor_SMD:C_0805_2012Metric_Pad1.18x1.45mm_HandSolder"
+		(property "Footprint" "PCM_Capacitor_SMD_AKL:C_0805_2012Metric_Pad1.18x1.45mm_HandSolder"
 			(at 200.66 92.71 0)
 			(effects
@@
 			)
 		)
-		(property "DigiKey" "311-1140-1-ND"
+		(property "DigiKey" ""
 			(at 200.66 92.71 0)
 			(effects
@@
 			)
 		)
-		(property "LCSC" "MBK0805X7R104K500NT"
+		(property "LCSC" "C1711"
 			(at 200.66 92.71 0)
 			(effects
